Commit message: Cart v1.0

File: universe/autoware.universe/launch/tier4_vehicle_launch/urdf/vehicle.xacro (robot description, xacro)
@@ -7,5 +7,6 @@
   <xacro:include filename="$(find ${vehicle_model_property}_description)/urdf/vehicle.xacro"/>
   <!-- sensors -->
-  <xacro:property name="sensor_model_property" value="$(arg sensor_model)"/>
-  <xacro:include filename="$(find ${sensor_model_property}_description)/urdf/sensors.xacro"/>
+  <!--HJK-->
+  <!-- <xacro:property name="sensor_model_property" value="$(arg sensor_model)"/>
+  <xacro:include filename="$(find ${sensor_model_property}_description)/urdf/sensors.xacro"/> -->
 </robot>

Commit message: feat(tier4_vehicle_launch): Removed sensors TF since too much useless TF is processed

File: universe/autoware.universe/launch/tier4_vehicle_launch/urdf/vehicle.xacro (robot description, xacro)
@@ -6,6 +6,3 @@
   <xacro:property name="vehicle_model_property" value="$(arg vehicle_model)"/>
   <xacro:include filename="$(find ${vehicle_model_property}_description)/urdf/vehicle.xacro"/>
-  <!-- sensors -->
-  <xacro:property name="sensor_model_property" value="$(arg sensor_model)"/>
-  <xacro:include filename="$(find ${sensor_model_property}_description)/urdf/sensors.xacro"/>
 </robot>

Commit message: comment: Add history to every commit

File: universe/autoware.universe/launch/tier4_vehicle_launch/urdf/vehicle.xacro (robot description, xacro)
@@ -6,3 +6,6 @@
   <xacro:property name="vehicle_model_property" value="$(arg vehicle_model)"/>
   <xacro:include filename="$(find ${vehicle_model_property}_description)/urdf/vehicle.xacro"/>
+  <!-- sensors -->
+  <!-- <xacro:property name="sensor_model_property" value="$(arg sensor_model)"/> --> <!--HJK_241126_C-->
+  <!-- <xacro:include filename="$(find ${sensor_model_property}_description)/urdf/sensors.xacro"/> --> <!--HJK_241126_C-->
 </robot>

Commit message: chg: disable(left&right)LiDAR in launch file

File: universe/autoware.universe/launch/tier4_vehicle_launch/urdf/vehicle.xacro (robot description, xacro)
@@ -6,6 +6,3 @@
   <xacro:property name="vehicle_model_property" value="$(arg vehicle_model)"/>
   <xacro:include filename="$(find ${vehicle_model_property}_description)/urdf/vehicle.xacro"/>
-  <!-- sensors -->
-  <!-- <xacro:property name="sensor_model_property" value="$(arg sensor_model)"/> --> <!--HJK_241126_C-->
-  <!-- <xacro:include filename="$(find ${sensor_model_property}_description)/urdf/sensors.xacro"/> --> <!--HJK_241126_C-->
 </robot>

Commit message: Fix : V1.0 for Niro

File: universe/autoware.universe/launch/tier4_vehicle_launch/urdf/vehicle.xacro (robot description, xacro)
@@ -6,3 +6,6 @@
   <xacro:property name="vehicle_model_property" value="$(arg vehicle_model)"/>
   <xacro:include filename="$(find ${vehicle_model_property}_description)/urdf/vehicle.xacro"/>
+  <!-- sensors
+  <xacro:property name="sensor_model_property" value="$(arg sensor_model)"/>
+  <xacro:include filename="$(find ${sensor_model_property}_description)/urdf/sensors.xacro"/> --> <!-- HJK_230000 --> <!-- TFs required are published separately (in launcher) -->
 </robot>
